Commit message: init commits for diana_hardware

File: diana_description/robots/diana7/diana7.ros2_control.xacro (robot description, xacro)
@@ -1,76 +1,85 @@
 <?xml version="1.0"?>
 <robot xmlns:xacro="http://www.ros.org/wiki/xacro">
-<xacro:macro
-    name="diana7_ros2_control"
-    params="
+    <xacro:macro
+        name="diana7_ros2_control"
+        params="
+        name:=DianaSystem
         prefix:=''
         use_fake_hardware:=true
-        fake_sensor_commands:=false
-    ">
-<ros2_control
-    name="${prefix}Diana7System"
-    type="system">
-    <hardware>
-        <xacro:if value="${use_fake_hardware}">
-            <plugin>
-                mock_components/GenericSystem
-            </plugin>
-            <param name="fake_sensor_commands">
-                ${fake_sensor_commands}
-            </param>
-            <param name="state_following_offset">
-                0.0
-            </param>
-        </xacro:if>
-        <xacro:unless value="${use_fake_hardware}">
-            <!-- 后续替换 -->
-            <plugin>
-                diana_hardware/DianaHardware
-            </plugin>
-        </xacro:unless>
-    </hardware>
-    <!-- joint1 -->
-    <joint name="${prefix}joint1">
-        <command_interface name="position"/>
-        <state_interface name="position"/>
-        <state_interface name="velocity"/>
-    </joint>
-    <!-- joint2 -->
-    <joint name="${prefix}joint2">
-        <command_interface name="position"/>
-        <state_interface name="position"/>
-        <state_interface name="velocity"/>
-    </joint>
-    <!-- joint3 -->
-    <joint name="${prefix}joint3">
-        <command_interface name="position"/>
-        <state_interface name="position"/>
-        <state_interface name="velocity"/>
-    </joint>
-    <!-- joint4 -->
-    <joint name="${prefix}joint4">
-        <command_interface name="position"/>
-        <state_interface name="position"/>
-        <state_interface name="velocity"/>
-    </joint>
-    <!-- joint5 -->
-    <joint name="${prefix}joint5">
-        <command_interface name="position"/>
-        <state_interface name="position"/>
-        <state_interface name="velocity"/>
-    </joint>
-    <!-- joint6 -->
-    <joint name="${prefix}joint6">
-        <command_interface name="position"/>
-        <state_interface name="position"/>
-        <state_interface name="velocity"/>
-    </joint>
-    <!-- joint7 -->
-    <joint name="${prefix}joint7">
-        <command_interface name="position"/>
-        <state_interface name="position"/>
-        <state_interface name="velocity"/>
-    </joint>
-</ros2_control>
-</xacro:macro>
+        robot_ip:=''
+        command_port:=1337
+        state_port:=1338
+        control_frequency:=1000">
+        <ros2_control name="${name}" type="system">
+            <hardware>
+                <plugin>
+                    diana_hardware/DianaSystem
+                </plugin>
+                <param name="use_fake_hardware">
+                    ${use_fake_hardware}
+                </param>
+                <param name="robot_ip">
+                    ${robot_ip}
+                </param>
+                <param name="command_port">
+                    ${command_port}
+                </param>
+                <param name="state_port">
+                    ${state_port}
+                </param>
+                <param name="control_frequency">
+                    ${control_frequency}
+                </param>
+            </hardware>
+            <!-- Joint 1 -->
+            <joint name="${prefix}joint1">
+                <command_interface name="position" />
+                <state_interface name="position" />
+                <state_interface name="velocity" />
+                <state_interface name="effort" />
+            </joint>
+            <!-- Joint 2 -->
+            <joint name="${prefix}joint2">
+                <command_interface name="position" />
+                <state_interface name="position" />
+                <state_interface name="velocity" />
+                <state_interface name="effort" />
+            </joint>
+            <!-- Joint 3 -->
+            <joint name="${prefix}joint3">
+                <command_interface name="position" />
+                <state_interface name="position" />
+                <state_interface name="velocity" />
+                <state_interface name="effort" />
+            </joint>
+            <!-- Joint 4 -->
+            <joint name="${prefix}joint4">
+                <command_interface name="position" />
+                <state_interface name="position" />
+                <state_interface name="velocity" />
+                <state_interface name="effort" />
+            </joint>
+            <!-- Joint 5 -->
+            <joint name="${prefix}joint5">
+                <command_interface name="position" />
+                <state_interface name="position" />
+                <state_interface name="velocity" />
+                <state_interface name="effort" />
+            </joint>
+            <!-- Joint 6 -->
+            <joint name="${prefix}joint6">
+                <command_interface name="position" />
+                <state_interface name="position" />
+                <state_interface name="velocity" />
+                <state_interface name="effort" />
+            </joint>
+            <!-- Joint 7 -->
+            <joint name="${prefix}joint7">
+                <command_interface name="position" />
+                <state_interface name="position" />
+                <state_interface name="velocity" />
+                <state_interface name="effort" />
+            </joint>
+        </ros2_control>
+    </xacro:macro>
 </robot>

File: diana_description/robots/diana7/diana7_robot.urdf.xacro (robot description, xacro)
@@ -1,2 +1,3 @@
+<?xml version="1.0"?>
 <robot name="diana7" xmlns:xacro="http://www.ros.org/wiki/xacro">
   <!-- ========= Arguments ========= -->
@@ -19,8 +20,13 @@
   <xacro:diana7 prefix="${prefix}"/>
   <!-- ========= ros2_control ========= -->
-  <xacro:diana7_ros2_control
-      prefix="${prefix}"
-      use_fake_hardware="$(arg use_fake_hardware)"
-      fake_sensor_commands="$(arg fake_sensor_commands)"/>
+<xacro:include filename="$(find diana_description)/robots/diana7/diana7.ros2_control.xacro"/>
+<xacro:diana7_ros2_control
+    name="DianaSystem"
+    prefix="${prefix}"
+    use_fake_hardware="${use_fake_hardware}"
+    robot_ip="${robot_ip}"
+    command_port="${command_port}"
+    state_port="${state_port}"
+    control_frequency="${control_frequency}"/>
   <!-- ========= Gazebo ========= -->
   <xacro:if value="$(arg use_gazebo)">
