Commit message: code updates on diana_description

File: diana_description/robots/diana7/diana7.urdf.xacro (robot description, xacro)
@@ -1,176 +1,67 @@
-<?xml version='1.0' encoding='utf-8'?>
-<robot xmlns:xacro="http://ros.org/wiki/xacro">
-  <xacro:macro name="dh_to_origin" params="a d alpha theta">
-    <xacro:property name="r00" scope="parent" value="${cos(theta)}" />
-    <xacro:property name="r10" scope="parent" value="${sin(theta)*cos(alpha)}" />
-    <xacro:property name="r11" scope="parent" value="${cos(theta)*cos(alpha)}" />
-    <xacro:property name="r12" scope="parent" value="${-sin(alpha)}" />
-    <xacro:property name="r20" scope="parent" value="${sin(theta)*sin(alpha)}" />
-    <xacro:property name="r21" scope="parent" value="${cos(theta)*sin(alpha)}" />
-    <xacro:property name="r22" scope="parent" value="${cos(alpha)}" />
-    <xacro:property name="sum" scope="parent" value="${sqrt(r00*r00 + r10*r10)}" />
-    <xacro:if value="${sum > 1e-15}">
-      <xacro:property name="ry" scope="parent" value="0.0" />
-      <xacro:property name="pitch0" scope="parent" value="${atan2(-r20,sum)}" />
-      <xacro:property name="pitch1" scope="parent" value="${atan2(-r20,-sum)}" />
-      <xacro:if value="${fabs(pitch0 - ry) > fabs(pitch1 - ry)}">
-        <origin rpy="${atan2(-r21,-r22)} ${pitch1} ${atan2(-r10,-r00)}"
-          xyz="${a} ${-sin(alpha)*d} ${cos(alpha)*d}" />
-      </xacro:if>
-      <xacro:unless value="${fabs(pitch0 - ry) > fabs(pitch1 - ry)}">
-        <origin rpy="${atan2(r21,r22)} ${pitch0} ${atan2(r10,r00)}"
-          xyz="${a} ${-sin(alpha)*d} ${cos(alpha)*d}" />
-      </xacro:unless>
-    </xacro:if>
-    <xacro:unless value="${sum > 1e-15}">
-      <origin rpy="${atan2(-r12,r11)} ${atan2(-r20,sum)} 0.0"
-        xyz="${a} ${-sin(alpha)*d} ${cos(alpha)*d}" />
-    </xacro:unless>
-  </xacro:macro>
-  <xacro:macro name="diana7"
-    params="prefix:='' safety_limits:=false safety_pos_margin:=0.15 safety_k_position:=20 safety_k_velocity:=0.0">
-    <xacro:property name="a" value="${[0.0,0.0,0.0,0.065,-0.0528,-0.0122,0.087]}" />
-    <xacro:property name="alpha"
-      value="${[3.1415926536,1.5707963267949,-1.5707963267949,1.5707963267949,-1.5707963267949,-1.5707963267949,-1.5707963267949]}" />
-    <xacro:property name="d" value="${[-0.2856,0.0,-0.4586,0.0,-0.4554,0.0,-0.1169]}" />
-    <xacro:property name="theta" value="${[0,0,0,0.0,0,3.1415926536,0]}" />
-    <xacro:property name="joint_limitU"
-      value="${[3.12413936107,1.5707963268,3.12413936107,3.05432619099,3.12413936107,3.12413936107,3.12413936107]}" />
-    <xacro:property name="joint_limitL"
-      value="${[-3.12413936107,-1.5707963268,-3.12413936107,0.0,-3.12413936107,-3.12413936107,-3.12413936107]}" />
-    <xacro:property name="joint_vel"
-      value="${[2.967059728,2.6179938780,2.6179938780,2.6179938780,3.14159265359,3.14159265359,3.839724354]}" />
-    <xacro:property name="joint_effort" value="${[235.0,235.0,111.0,111.0,54.0,54.0,54.0]}" />
-    <xacro:property name="link1_rbi"
-      value="${[5.299828,-0.000017,0.000007,0.033580,0.029705,-3.9e-05,-2.4e-05,0.02688,-7e-05,0.015918]}" />
-    <xacro:property name="link2_rbi"
-      value="${[3.246370,-0.000015,-0.046026,-0.035713,0.020388,-2e-06,-0.0,0.009309,0.005307,0.01893]}" />
-    <xacro:property name="link3_rbi"
-      value="${[5.231815,0.027041,0.001592,0.140231,0.117623,-0.000425,0.021147,0.121236,0.001127,0.019132]}" />
-    <xacro:property name="link4_rbi"
-      value="${[1.940060,-0.026110,-0.042551,-0.029657,0.009292,-0.002304,0.001465,0.005983,0.002463,0.009392]}" />
-    <xacro:property name="link5_rbi"
-      value="${[2.678626,-0.006541,0.023619,0.193770,0.063743,0.000512,-0.002363,0.061192,0.008513,0.006265]}" />
-    <xacro:property name="link6_rbi"
-      value="${[2.856811,0.048158,-0.015440,0.001272,0.007152,0.001764,0.000167,0.010739,-5.3e-05,0.011456]}" />
-    <xacro:property name="link7_rbi"
-      value="${[0.575995,0.000488,0.000000,0.038260,0.000876,0.0,6e-06,0.000891,0.0,0.000481]}" />
-    <xacro:property name="joint_damp" value="0.0" />
-    <xacro:property name="joint_frict" value="0.1" />
-    <link name="${prefix}base_link">
-      <inertial>
-        <origin rpy="0 0 0" xyz="0.0 0.0 0.0" />
-        <mass value="5.0" />
-        <inertia ixx="0.0" ixy="0.0" ixz="0.0" iyy="0.0" iyz="0.0" izz="0.0" />
-      </inertial>
-      <visual>
-        <origin rpy="0 0 0" xyz="0 0 0" />
-        <geometry>
-          <mesh filename="package://diana_description/meshes/base_link.STL" />
-        </geometry>
-        <material name="LightGrey">
-          <color rgba="0.7 0.7 0.7 1" />
-        </material>
-      </visual>
-      <collision>
-        <origin rpy="0 0 0" xyz="0 0 0" />
-        <geometry>
-          <mesh filename="package://diana_description/meshes/base_link.STL" />
-        </geometry>
-      </collision>
-    </link>
-    <link name="${prefix}tool0" />
-    <joint name="${prefix}tool0_fixed" type="fixed">
-      <parent link="${prefix}link7" />
-      <child link="${prefix}tool0" />
-    </joint>
-    <xacro:macro name="add_joint" params="num a alpha d theta limitU limitL vel effort">
-      <xacro:if value="${num == 1}">
-        <xacro:property name="parent_link" value="${prefix}base_link" />
-      </xacro:if>
-      <xacro:unless value="${num == 1}">
-        <xacro:property name="parent_link" value="${prefix}link${num-1}" />
-      </xacro:unless>
-      <joint name="${prefix}joint${num}" type="revolute">
-        <xacro:dh_to_origin a="${a}" alpha="${alpha}" d="${d}" theta="${theta}" />
-        <parent link="${parent_link}" />
-        <child link="${prefix}link${num}" />
-        <axis xyz="0 0 1" />
-        <limit effort="${effort}" lower="${limitL}" upper="${limitU}" velocity="${vel}" />
-        <xacro:if value="${safety_limits}">
-          <safety_controller k_position="${safety_k_position}" k_velocity="${safety_k_velocity}"
-            soft_lower_limit="${limitL + safety_pos_margin}"
-            soft_upper_limit="${limitU - safety_pos_margin}" />
-        </xacro:if>
-        <dynamics damping="${joint_damp}" friction="${joint_frict}" />
-      </joint>
-    </xacro:macro>
-    <xacro:add_joint a="${a[0]}" alpha="${alpha[0]}" d="${d[0]}" effort="${joint_effort[0]}"
-      limitL="${joint_limitL[0]}" limitU="${joint_limitU[0]}" num="1" theta="${theta[0]}"
-      vel="${joint_vel[0]}" />
-    <xacro:add_joint a="${a[1]}" alpha="${alpha[1]}" d="${d[1]}" effort="${joint_effort[1]}"
-      limitL="${joint_limitL[1]}" limitU="${joint_limitU[1]}" num="2" theta="${theta[1]}"
-      vel="${joint_vel[1]}" />
-    <xacro:add_joint a="${a[2]}" alpha="${alpha[2]}" d="${d[2]}" effort="${joint_effort[2]}"
-      limitL="${joint_limitL[2]}" limitU="${joint_limitU[2]}" num="3" theta="${theta[2]}"
-      vel="${joint_vel[2]}" />
-    <xacro:add_joint a="${a[3]}" alpha="${alpha[3]}" d="${d[3]}" effort="${joint_effort[3]}"
-      limitL="${joint_limitL[3]}" limitU="${joint_limitU[3]}" num="4" theta="${theta[3]}"
-      vel="${joint_vel[3]}" />
-    <xacro:add_joint a="${a[4]}" alpha="${alpha[4]}" d="${d[4]}" effort="${joint_effort[4]}"
-      limitL="${joint_limitL[4]}" limitU="${joint_limitU[4]}" num="5" theta="${theta[4]}"
-      vel="${joint_vel[4]}" />
-    <xacro:add_joint a="${a[5]}" alpha="${alpha[5]}" d="${d[5]}" effort="${joint_effort[5]}"
-      limitL="${joint_limitL[5]}" limitU="${joint_limitU[5]}" num="6" theta="${theta[5]}"
-      vel="${joint_vel[5]}" />
-    <xacro:add_joint a="${a[6]}" alpha="${alpha[6]}" d="${d[6]}" effort="${joint_effort[6]}"
-      limitL="${joint_limitL[6]}" limitU="${joint_limitU[6]}" num="7" theta="${theta[6]}"
-      vel="${joint_vel[6]}" />
-    <xacro:macro name="add_link" params="num mass x y z ixx ixy ixz iyy iyz izz">
-      <link name="${prefix}link${num}">
-        <inertial>
-          <origin rpy="0 0 0" xyz="${x} ${y} ${z}" />
-          <mass value="${mass}" />
-          <inertia ixx="${ixx}" ixy="${ixy}" ixz="${ixz}" iyy="${iyy}" iyz="${iyz}" izz="${izz}" />
-        </inertial>
-        <visual>
-          <origin rpy="0 0 0" xyz="0 0 0" />
-          <geometry>
-            <mesh filename="package://diana_description/meshes/link${num}.STL" />
-          </geometry>
-          <material name="LightGrey">
-            <color rgba="0.7 0.7 0.7 1" />
-          </material>
-        </visual>
-        <collision>
-          <origin rpy="0 0 0" xyz="0 0 0" />
-          <geometry>
-            <mesh filename="package://diana_description/meshes/link${num}.STL" />
-          </geometry>
-        </collision>
-      </link>
-    </xacro:macro>
-    <xacro:add_link ixx="${link1_rbi[4]}" ixy="${link1_rbi[5]}" ixz="${link1_rbi[6]}"
-      iyy="${link1_rbi[7]}" iyz="${link1_rbi[8]}" izz="${link1_rbi[9]}" mass="${link1_rbi[0]}"
-      num="1" x="${link1_rbi[1]}" y="${link1_rbi[2]}" z="${link1_rbi[3]}" />
-    <xacro:add_link ixx="${link2_rbi[4]}" ixy="${link2_rbi[5]}" ixz="${link2_rbi[6]}"
-      iyy="${link2_rbi[7]}" iyz="${link2_rbi[8]}" izz="${link2_rbi[9]}" mass="${link2_rbi[0]}"
-      num="2" x="${link2_rbi[1]}" y="${link2_rbi[2]}" z="${link2_rbi[3]}" />
-    <xacro:add_link ixx="${link3_rbi[4]}" ixy="${link3_rbi[5]}" ixz="${link3_rbi[6]}"
-      iyy="${link3_rbi[7]}" iyz="${link3_rbi[8]}" izz="${link3_rbi[9]}" mass="${link3_rbi[0]}"
-      num="3" x="${link3_rbi[1]}" y="${link3_rbi[2]}" z="${link3_rbi[3]}" />
-    <xacro:add_link ixx="${link4_rbi[4]}" ixy="${link4_rbi[5]}" ixz="${link4_rbi[6]}"
-      iyy="${link4_rbi[7]}" iyz="${link4_rbi[8]}" izz="${link4_rbi[9]}" mass="${link4_rbi[0]}"
-      num="4" x="${link4_rbi[1]}" y="${link4_rbi[2]}" z="${link4_rbi[3]}" />
-    <xacro:add_link ixx="${link5_rbi[4]}" ixy="${link5_rbi[5]}" ixz="${link5_rbi[6]}"
-      iyy="${link5_rbi[7]}" iyz="${link5_rbi[8]}" izz="${link5_rbi[9]}" mass="${link5_rbi[0]}"
-      num="5" x="${link5_rbi[1]}" y="${link5_rbi[2]}" z="${link5_rbi[3]}" />
-    <xacro:add_link ixx="${link6_rbi[4]}" ixy="${link6_rbi[5]}" ixz="${link6_rbi[6]}"
-      iyy="${link6_rbi[7]}" iyz="${link6_rbi[8]}" izz="${link6_rbi[9]}" mass="${link6_rbi[0]}"
-      num="6" x="${link6_rbi[1]}" y="${link6_rbi[2]}" z="${link6_rbi[3]}" />
-    <xacro:add_link ixx="${link7_rbi[4]}" ixy="${link7_rbi[5]}" ixz="${link7_rbi[6]}"
-      iyy="${link7_rbi[7]}" iyz="${link7_rbi[8]}" izz="${link7_rbi[9]}" mass="${link7_rbi[0]}"
-      num="7" x="${link7_rbi[1]}" y="${link7_rbi[2]}" z="${link7_rbi[3]}" />
-    <xacro:diana7_arm_gazebo />
-  </xacro:macro>
+<?xml version="1.0"?>
+<robot
+    xmlns:xacro="http://www.ros.org/wiki/xacro"
+    name="diana7">
+  <!-- ====================================================== -->
+  <!-- Arguments                                               -->
+  <!-- ====================================================== -->
+  <xacro:arg name="prefix" default=""/>
+  <xacro:arg name="use_fake_hardware" default="true"/>
+  <xacro:arg name="fake_sensor_commands" default="false"/>
+  <xacro:arg name="use_gazebo" default="false"/>
+  <xacro:arg name="robot_ip" default=""/>
+  <xacro:arg name="command_port" default="1337"/>
+  <xacro:arg name="state_port" default="1338"/>
+  <xacro:arg name="control_frequency" default="1000"/>
+  <!-- ====================================================== -->
+  <!-- Properties                                              -->
+  <!-- ====================================================== -->
+  <xacro:property name="prefix"
+                  value="$(arg prefix)"/>
+  <xacro:property name="use_fake_hardware"
+                  value="$(arg use_fake_hardware)"/>
+  <xacro:property name="fake_sensor_commands"
+                  value="$(arg fake_sensor_commands)"/>
+  <xacro:property name="use_gazebo"
+                  value="$(arg use_gazebo)"/>
+  <xacro:property name="robot_ip"
+                  value="$(arg robot_ip)"/>
+  <xacro:property name="command_port"
+                  value="$(arg command_port)"/>
+  <xacro:property name="state_port"
+                  value="$(arg state_port)"/>
+  <xacro:property name="control_frequency"
+                  value="$(arg control_frequency)"/>
+  <!-- ====================================================== -->
+  <!-- Includes                                                -->
+  <!-- ====================================================== -->
+  <xacro:include
+      filename="$(find diana_description)/robots/diana7/diana7_arm.urdf.xacro"/>
+  <xacro:include
+      filename="$(find diana_description)/robots/diana7/diana7.ros2_control.xacro"/>
+  <xacro:include
+      filename="$(find diana_description)/robots/diana7/diana7.gazebo.xacro"/>
+  <!-- ====================================================== -->
+  <!-- Robot                                                   -->
+  <!-- ====================================================== -->
+  <xacro:diana7
+      prefix="${prefix}"/>
+  <!-- ====================================================== -->
+  <!-- ros2_control                                            -->
+  <!-- ====================================================== -->
+  <xacro:diana7_ros2_control
+      name="DianaSystem"
+      prefix="${prefix}"
+      use_fake_hardware="${use_fake_hardware}"
+      robot_ip="${robot_ip}"
+      command_port="${command_port}"
+      state_port="${state_port}"
+      control_frequency="${control_frequency}"/>
+  <!-- ====================================================== -->
+  <!-- Gazebo                                                  -->
+  <!-- ====================================================== -->
+  <xacro:if value="${use_gazebo}">
+    <xacro:diana7_gazebo
+        prefix="${prefix}"/>
+  </xacro:if>
 </robot>
